File: KiCad_Project/3DProUsb.sch (KiCad schematic (older format))
At the start: 24 parts, among them J1 USB_B_Micro, J2 AVR_Program, J3 DA15-SL-25, SW1 SW_Push_Dual, U1 ATMEGA32U4-MU, X1 16MHz

Commit message: Turned top layer into additional ground plane and added no connect labels to unused clock pins
Connections:
- no-connect marks 26 -> 28
Changed lines of the file:
@@
 NoConn ~ 7350 2550
 NoConn ~ 6950 2350
+NoConn ~ 7500 3050
+NoConn ~ 8100 3050
 $EndSCHEMATC

Commit message: Corrected USB port error
Parts:
- removed J1: USB_B_Micro, USB:MOLEX_1050170001, symbol Connector:USB_B_Micro
- added J1: 105164-0001, USB:MOLEX_105164-0001, symbol USB:105164-0001
Connections:
- net Earth: now also J1.5
- net VCC: now also J1.1
- net at R2.2: now also J1.2
- net at R1.2: now also J1.3
- no-connect marks 28 -> 33
Changed lines of the file:
@@
 L power:Earth #PWR0101
 U 1 1 5F49F689
-P 1650 3750
-F 0 "#PWR0101" H 1650 3500 50  0001 C CNN
-F 1 "Earth" H 1650 3600 50  0001 C CNN
-F 2 "" H 1650 3750 50  0001 C CNN
-F 3 "~" H 1650 3750 50  0001 C CNN
-	1    1650 3750
+P 1800 3650
+F 0 "#PWR0101" H 1800 3400 50  0001 C CNN
+F 1 "Earth" H 1800 3500 50  0001 C CNN
+F 2 "" H 1800 3650 50  0001 C CNN
+F 3 "~" H 1800 3650 50  0001 C CNN
+	1    1800 3650
 	1    0    0    -1
 $EndComp
@@
 	1    0    0    -1
 $EndComp
-Wire Wire Line
-	1650 3650 1650 3750
 $Comp
 L power:Earth #PWR0108
@@
 $EndComp
 NoConn ~ 7450 4500
-NoConn ~ 1950 3450
-NoConn ~ 1550 3650
 NoConn ~ 7450 4600
 NoConn ~ 7450 4800
-Wire Wire Line
-	1950 3250 2250 3250
 Wire Wire Line
 	1950 3350 2850 3350
@@
 NoConn ~ 3450 4550
 NoConn ~ 3450 4850
-Wire Wire Line
-	1950 3050 2050 3050
 Wire Wire Line
 	2050 3050 2050 2100
@@
 	1850 4000 1850 4250
 $Comp
-L Connector:USB_B_Micro J1
-U 1 1 5F48D0F5
-P 1650 3250
-F 0 "J1" H 1707 3717 50  0000 C CNN
-F 1 "USB_B_Micro" H 1707 3626 50  0000 C CNN
-F 2 "USB:MOLEX_1050170001" H 1800 3200 50  0001 C CNN
-F 3 "~" H 1800 3200 50  0001 C CNN
-F 4 "1051640001" H 1650 3250 50  0001 C CNN "ManufacturerPart"
-F 5 "WM11263CT-ND" H 1650 3250 50  0001 C CNN "DigikeyPart"
-	1    1650 3250
-	1    0    0    -1
-$EndComp
-$Comp
 L Connector_Generic:Conn_02x03_Odd_Even J2
 U 1 1 5F814BD5
@@
 NoConn ~ 7500 3050
 NoConn ~ 8100 3050
+$Comp
+L USB:105164-0001 J1
+U 1 1 5F69BCA2
+P 1250 3350
+F 0 "J1" H 1143 3917 50  0000 C CNN
+F 1 "105164-0001" H 1143 3826 50  0000 C CNN
+F 2 "USB:MOLEX_105164-0001" H 1250 3350 50  0001 L BNN
+F 3 "molex" H 1250 3350 50  0001 L BNN
+F 4 "B" H 1250 3350 50  0001 L BNN "Field4"
+F 5 "Manufacturer recommendations" H 1250 3350 50  0001 L BNN "Field5"
+F 6 "1051640001" H 1250 3350 50  0001 C CNN "ManufacturerPart"
+F 7 "WM11263CT-ND" H 1250 3350 50  0001 C CNN "DigikeyPart"
+	1    1250 3350
+	-1   0    0    -1
+$EndComp
+Wire Wire Line
+	1650 3050 2050 3050
+Wire Wire Line
+	1650 3250 2250 3250
+Wire Wire Line
+	1950 3350 1950 3150
+Wire Wire Line
+	1950 3150 1650 3150
+Wire Wire Line
+	1650 3450 1800 3450
+Wire Wire Line
+	1800 3450 1800 3650
+NoConn ~ 1650 3350
+NoConn ~ 1650 3650
+NoConn ~ 1650 3750
+NoConn ~ 1650 3850
+NoConn ~ 1650 3950
+NoConn ~ 1650 4050
+NoConn ~ 1650 4150
 $EndSCHEMATC

Commit message: Connected ground pins of clock
Connections:
- net Earth: now also X1.2 (GND), X1.4 (V+)
- no-connect marks 33 -> 31
Changed lines of the file:
@@
 U 1 1 5F53A5CC
 P 7800 3050
-F 0 "X1" V 7754 3394 50  0000 L CNN
-F 1 "16MHz" V 7845 3394 50  0000 L CNN
+F 0 "X1" V 7600 3350 50  0000 L CNN
+F 1 "16MHz" V 7700 3350 50  0000 L CNN
 F 2 "Oscillator:Oscillator_SMD_SeikoEpson_SG8002CE-4Pin_3.2x2.5mm" H 8500 2700 50  0001 C CNN
 F 3 "http://cdn-reichelt.de/documents/datenblatt/B400/XO91.pdf" H 7700 3050 50  0001 C CNN
@@
 NoConn ~ 7350 2550
 NoConn ~ 6950 2350
-NoConn ~ 7500 3050
-NoConn ~ 8100 3050
 $Comp
 L USB:105164-0001 J1
@@
 NoConn ~ 1650 4050
 NoConn ~ 1650 4150
+$Comp
+L power:Earth #PWR?
+U 1 1 5F6D414B
+P 7400 3150
+F 0 "#PWR?" H 7400 2900 50  0001 C CNN
+F 1 "Earth" H 7400 3000 50  0001 C CNN
+F 2 "" H 7400 3150 50  0001 C CNN
+F 3 "~" H 7400 3150 50  0001 C CNN
+	1    7400 3150
+	1    0    0    -1
+$EndComp
+$Comp
+L power:Earth #PWR?
+U 1 1 5F6D5453
+P 8200 3100
+F 0 "#PWR?" H 8200 2850 50  0001 C CNN
+F 1 "Earth" H 8200 2950 50  0001 C CNN
+F 2 "" H 8200 3100 50  0001 C CNN
+F 3 "~" H 8200 3100 50  0001 C CNN
+	1    8200 3100
+	1    0    0    -1
+$EndComp
+Wire Wire Line
+	7500 3050 7400 3050
+Wire Wire Line
+	7400 3050 7400 3150
+Wire Wire Line
+	8100 3050 8200 3050
+Wire Wire Line
+	8200 3050 8200 3100
 $EndSCHEMATC

Commit message: Added missing component and connections
Parts:
- added C11: 1uF, Capacitor_SMD:C_0402_1005Metric, symbol Device:CP1_Small
Connections:
- net Earth: now also C11.2
- net VCC: no longer U1.6 (UCAP)
- net PB0_PD0: now reaches U1.18 ((OC0B/SCL/INT0)PD0)
- net PB0_PD0: now also J3.2, U1.8 ((SS/PCINT0)PB0)
- new net: C11.1, U1.6 (UCAP)
- no-connect marks 31 -> 30
Other:
- moved on the sheet: C3, C4, C5
Changed lines of the file:
@@
 L Device:CP1_Small C3
 U 1 1 5F4ADDE0
-P 2000 5300
-F 0 "C3" H 2091 5346 50  0000 L CNN
-F 1 "0.1uF" H 2091 5255 50  0000 L CNN
-F 2 "Capacitor_SMD:C_0402_1005Metric" H 2000 5300 50  0001 C CNN
-F 3 "~" H 2000 5300 50  0001 C CNN
-F 4 "TMK105B7104KV-FR" H 2000 5300 50  0001 C CNN "ManufacturerPart"
-F 5 "587-5476-1-ND" H 2000 5300 50  0001 C CNN "DigikeyPart"
-	1    2000 5300
+P 2000 5100
+F 0 "C3" H 2091 5146 50  0000 L CNN
+F 1 "0.1uF" H 2091 5055 50  0000 L CNN
+F 2 "Capacitor_SMD:C_0402_1005Metric" H 2000 5100 50  0001 C CNN
+F 3 "~" H 2000 5100 50  0001 C CNN
+F 4 "TMK105B7104KV-FR" H 2000 5100 50  0001 C CNN "ManufacturerPart"
+F 5 "587-5476-1-ND" H 2000 5100 50  0001 C CNN "DigikeyPart"
+	1    2000 5100
 	1    0    0    -1
 $EndComp
@@
 L Device:CP1_Small C4
 U 1 1 5F4B5EC5
-P 1600 5300
-F 0 "C4" H 1691 5346 50  0000 L CNN
-F 1 "0.1uF" H 1691 5255 50  0000 L CNN
-F 2 "Capacitor_SMD:C_0402_1005Metric" H 1600 5300 50  0001 C CNN
-F 3 "~" H 1600 5300 50  0001 C CNN
-F 4 "TMK105B7104KV-FR" H 1600 5300 50  0001 C CNN "ManufacturerPart"
-F 5 "587-5476-1-ND" H 1600 5300 50  0001 C CNN "DigikeyPart"
-	1    1600 5300
+P 1600 5100
+F 0 "C4" H 1691 5146 50  0000 L CNN
+F 1 "0.1uF" H 1691 5055 50  0000 L CNN
+F 2 "Capacitor_SMD:C_0402_1005Metric" H 1600 5100 50  0001 C CNN
+F 3 "~" H 1600 5100 50  0001 C CNN
+F 4 "TMK105B7104KV-FR" H 1600 5100 50  0001 C CNN "ManufacturerPart"
+F 5 "587-5476-1-ND" H 1600 5100 50  0001 C CNN "DigikeyPart"
+	1    1600 5100
 	1    0    0    -1
 $EndComp
@@
 L Device:CP1_Small C5
 U 1 1 5F4B74CB
-P 1200 5300
-F 0 "C5" H 1291 5346 50  0000 L CNN
-F 1 "0.1uF" H 1291 5255 50  0000 L CNN
-F 2 "Capacitor_SMD:C_0402_1005Metric" H 1200 5300 50  0001 C CNN
-F 3 "~" H 1200 5300 50  0001 C CNN
-F 4 "TMK105B7104KV-FR" H 1200 5300 50  0001 C CNN "ManufacturerPart"
-F 5 "587-5476-1-ND" H 1200 5300 50  0001 C CNN "DigikeyPart"
-	1    1200 5300
+P 1200 5100
+F 0 "C5" H 1291 5146 50  0000 L CNN
+F 1 "0.1uF" H 1291 5055 50  0000 L CNN
+F 2 "Capacitor_SMD:C_0402_1005Metric" H 1200 5100 50  0001 C CNN
+F 3 "~" H 1200 5100 50  0001 C CNN
+F 4 "TMK105B7104KV-FR" H 1200 5100 50  0001 C CNN "ManufacturerPart"
+F 5 "587-5476-1-ND" H 1200 5100 50  0001 C CNN "DigikeyPart"
+	1    1200 5100
 	1    0    0    -1
 $EndComp
@@
 L power:Earth #PWR0104
 U 1 1 5F4BBC26
-P 1200 5600
-F 0 "#PWR0104" H 1200 5350 50  0001 C CNN
-F 1 "Earth" H 1200 5450 50  0001 C CNN
-F 2 "" H 1200 5600 50  0001 C CNN
-F 3 "~" H 1200 5600 50  0001 C CNN
-	1    1200 5600
+P 1200 5400
+F 0 "#PWR0104" H 1200 5150 50  0001 C CNN
+F 1 "Earth" H 1200 5250 50  0001 C CNN
+F 2 "" H 1200 5400 50  0001 C CNN
+F 3 "~" H 1200 5400 50  0001 C CNN
+	1    1200 5400
 	1    0    0    -1
 $EndComp
@@
 L power:Earth #PWR0105
 U 1 1 5F4BC419
-P 1600 5600
-F 0 "#PWR0105" H 1600 5350 50  0001 C CNN
-F 1 "Earth" H 1600 5450 50  0001 C CNN
-F 2 "" H 1600 5600 50  0001 C CNN
-F 3 "~" H 1600 5600 50  0001 C CNN
-	1    1600 5600
+P 1600 5400
+F 0 "#PWR0105" H 1600 5150 50  0001 C CNN
+F 1 "Earth" H 1600 5250 50  0001 C CNN
+F 2 "" H 1600 5400 50  0001 C CNN
+F 3 "~" H 1600 5400 50  0001 C CNN
+	1    1600 5400
 	1    0    0    -1
 $EndComp
@@
 L power:Earth #PWR0106
 U 1 1 5F4BCB40
-P 2000 5600
-F 0 "#PWR0106" H 2000 5350 50  0001 C CNN
-F 1 "Earth" H 2000 5450 50  0001 C CNN
-F 2 "" H 2000 5600 50  0001 C CNN
-F 3 "~" H 2000 5600 50  0001 C CNN
-	1    2000 5600
-	1    0    0    -1
-$EndComp
-Wire Wire Line
-	2000 5400 2000 5600
-Wire Wire Line
-	1600 5400 1600 5600
-Wire Wire Line
-	1200 5400 1200 5600
+P 2000 5400
+F 0 "#PWR0106" H 2000 5150 50  0001 C CNN
+F 1 "Earth" H 2000 5250 50  0001 C CNN
+F 2 "" H 2000 5400 50  0001 C CNN
+F 3 "~" H 2000 5400 50  0001 C CNN
+	1    2000 5400
+	1    0    0    -1
+$EndComp
+Wire Wire Line
+	2000 5200 2000 5400
+Wire Wire Line
+	1600 5200 1600 5400
+Wire Wire Line
+	1200 5200 1200 5400
 $Comp
 L power:Earth #PWR0107
@@
 NoConn ~ 3450 3550
 NoConn ~ 3450 3650
-NoConn ~ 3450 3850
 NoConn ~ 3450 3950
 NoConn ~ 3450 4050
@@
 Wire Wire Line
 	3350 2950 3350 3050
-Wire Wire Line
-	3350 5050 3450 5050
 Connection ~ 3350 3050
 Wire Wire Line
-	3350 5050 2000 5050
-Wire Wire Line
-	2000 5050 2000 5200
-Connection ~ 3350 5050
-Wire Wire Line
-	1600 5050 1600 5200
-Connection ~ 2000 5050
-Wire Wire Line
-	1600 5050 1200 5050
-Wire Wire Line
-	1200 5050 1200 5200
-Connection ~ 1600 5050
+	3350 4850 2000 4850
+Wire Wire Line
+	2000 4850 2000 5000
+Wire Wire Line
+	1600 4850 1600 5000
+Connection ~ 2000 4850
+Wire Wire Line
+	1600 4850 1200 4850
+Wire Wire Line
+	1200 4850 1200 5000
+Connection ~ 1600 4850
 Text GLabel 3500 1750 2    50   Input ~ 0
 VCC
@@
 	3200 5350 3200 5450
 Wire Wire Line
-	2000 5050 1600 5050
+	2000 4850 1600 4850
 $Comp
 L Device:R_US R3
@@
 	8550 2750 8700 2750
 Wire Wire Line
-	6250 3450 7350 3450
+	6250 3450 6800 3450
 Wire Wire Line
 	7350 4200 7450 4200
@@
 	2550 3250 3450 3250
 Wire Wire Line
-	3350 3050 3350 5050
+	3350 3050 3350 4850
 $Comp
 L Atmel:ATMEGA32U4-MU U1
@@
 Wire Wire Line
 	8200 3050 8200 3100
+Text GLabel 6300 2150 0    50   Input ~ 0
+PB0_PD0
+Text GLabel 3200 3850 0    50   Input ~ 0
+PB0_PD0
+Wire Wire Line
+	3200 3850 3450 3850
+Wire Wire Line
+	6300 2150 6800 2150
+Wire Wire Line
+	6800 2150 6800 3450
+Connection ~ 6800 3450
+Wire Wire Line
+	6800 3450 7350 3450
+$Comp
+L Device:CP1_Small C11
+U 1 1 5F92B196
+P 2500 5300
+F 0 "C11" H 2591 5346 50  0000 L CNN
+F 1 "1uF" H 2591 5255 50  0000 L CNN
+F 2 "Capacitor_SMD:C_0402_1005Metric" H 2500 5300 50  0001 C CNN
+F 3 "~" H 2500 5300 50  0001 C CNN
+F 4 "EMK105BJ105KV-F" H 2500 5300 50  0001 C CNN "ManufacturerPart"
+F 5 "587-2477-1-ND" H 2500 5300 50  0001 C CNN "DigiKeyPart"
+	1    2500 5300
+	1    0    0    -1
+$EndComp
+Wire Wire Line
+	3450 5050 2500 5050
+Wire Wire Line
+	2500 5050 2500 5200
+$Comp
+L power:Earth #PWR?
+U 1 1 5F93972C
+P 2500 5550
+F 0 "#PWR?" H 2500 5300 50  0001 C CNN
+F 1 "Earth" H 2500 5400 50  0001 C CNN
+F 2 "" H 2500 5550 50  0001 C CNN
+F 3 "~" H 2500 5550 50  0001 C CNN
+	1    2500 5550
+	1    0    0    -1
+$EndComp
+Wire Wire Line
+	2500 5400 2500 5550
 $EndSCHEMATC

Commit message: New board layout.  Made things smaller, removed large trenches, and calculated USB differential impedance.
Parts:
- removed J1: 105164-0001, USB:MOLEX_105164-0001, symbol USB:105164-0001
- added J1: 10118193-0001LF, USB:FCI_10118193-0001LF, symbol USB:10118193-0001LF
Changed lines of the file:
@@
 NoConn ~ 7350 2550
 NoConn ~ 6950 2350
-$Comp
-L USB:105164-0001 J1
-U 1 1 5F69BCA2
-P 1250 3350
-F 0 "J1" H 1143 3917 50  0000 C CNN
-F 1 "105164-0001" H 1143 3826 50  0000 C CNN
-F 2 "USB:MOLEX_105164-0001" H 1250 3350 50  0001 L BNN
-F 3 "molex" H 1250 3350 50  0001 L BNN
-F 4 "B" H 1250 3350 50  0001 L BNN "Field4"
-F 5 "Manufacturer recommendations" H 1250 3350 50  0001 L BNN "Field5"
-F 6 "1051640001" H 1250 3350 50  0001 C CNN "ManufacturerPart"
-F 7 "WM11263CT-ND" H 1250 3350 50  0001 C CNN "DigikeyPart"
-	1    1250 3350
-	-1   0    0    -1
-$EndComp
 Wire Wire Line
 	1650 3050 2050 3050
@@
 Wire Wire Line
 	2500 5400 2500 5550
+$Comp
+L USB:10118193-0001LF J1
+U 1 1 5F939EA9
+P 1250 3350
+F 0 "J1" H 1143 3915 50  0000 C CNN
+F 1 "10118193-0001LF" H 1143 3824 50  0000 C CNN
+F 2 "USB:FCI_10118193-0001LF" H 1250 3350 50  0001 L BNN
+F 3 "None" H 1250 3350 50  0001 L BNN
+F 4 "10118193-0001LF" H 1250 3350 50  0001 L BNN "Field4"
+F 5 "Single Port 5 Contact Shielded SMT MICRO USB B-Type Receptacle" H 1250 3350 50  0001 L BNN "Field5"
+F 6 "Amphenol FCI" H 1250 3350 50  0001 L BNN "Field6"
+F 7 "None" H 1250 3350 50  0001 L BNN "Field7"
+F 8 "Unavailable" H 1250 3350 50  0001 L BNN "Field8"
+F 9 "10118193-0001LF" H 1250 3350 50  0001 C CNN "ManufacturerPart"
+F 10 "609-4616-2-ND" H 1250 3350 50  0001 C CNN "DigiKeyPart"
+	1    1250 3350
+	-1   0    0    -1
+$EndComp
 $EndSCHEMATC
